Commit message: CI

File: vendor/robots/universal_robot/ur_description/ur5_camera.urdf (robot description, URDF)
Before this commit: robot ur5_camera, 9 links, 8 joints
Links:
- removed link end_effector
- added link ee_link, mass 0.0; collision box size=0 0 0
- link wrist_3_link: geometry collision mesh filename=meshes/collision/wrist3.stl; visual mesh filename=meshes/visual/wrist3.stl
Joints:
- removed joint wrist_3__fixed_joint__end_effector
- added joint ee_joint: type fixed, parent wrist_3_link, child ee_link, origin xyz=0 0.0823 0 rpy=0 0 0
- joint camera_joint: origin xyz=0 0.08 0.04 rpy=2.0943951023931953 3.141592653589793 0 -> xyz=0 -0.01 0.06 rpy=2.0943951023931953 3.141592653589793 3.141592653589793; parent end_effector -> ee_link
- joint shoulder_pan_joint: origin xyz=0.0 0.0 0.089159 rpy=0.0 0.0 3.141592653589793 -> xyz=0.0 0.0 0.089159 rpy=0.0 0.0 0.0
