Commit message: Implemented cartesian position controller.

File: coffee/models/vendor/robot_arms/kuka/iiwa_description/urdf/iiwa14_polytope_collision.urdf (robot description, URDF)
Before this commit: robot iiwa14, 11 links, 10 joints
Links:
- removed link base
- removed link iiwa_link_ee
- removed link iiwa_link_ee_kuka
- added link ee_link, mass 0.0; collision box size=0 0 0
- added link world
Joints:
- removed joint iiwa_joint_ee
- removed joint tool0_joint
- added joint ee_fixed_joint: type fixed, parent iiwa_link_7, child ee_link, origin xyz=0.0 0.0 0.045 rpy=3.141592653589793 0 0
- joint iiwa_base_joint: parent base -> world

File: coffee/models/vendor/robot_arms/ufactory/xarm7_description/xarm7.urdf (robot description, URDF)
Before this commit: robot xarm7, 10 links, 9 joints
Joints:
- joint ee_fixed_joint: origin xyz=0.0 0.0 0.0 rpy=0.0 0.0 0 -> xyz=0.0 0.0 0.0 rpy=0 3.141592653589793 3.141592653589793

File: coffee/models/vendor/robot_arms/universal_robot/ur5_description/ur5.urdf (robot description, URDF)
Before this commit: robot universal_robot, 8 links, 7 joints
Joints:
- joint ee_joint: origin xyz=0 0.0823 0 rpy=0 0 0 -> xyz=0 0.0823 0 rpy=1.57079632679 -1.57079632679 0
