Commit message: Prelim implementation of robot composition (arm + gripper).

File: coffee/models/vendor/end_effectors/schunk/wsg_50_description/model.urdf (robot description, URDF)
Before this commit: robot wsg_50, 5 links, 4 joints
Links:
- added link pinch_site, mass 0.0; collision box size=0 0 0; visual box size=0.01 0.01 0.01
Joints:
- added joint tcp_joint: type fixed, parent wsg_base_link, child pinch_site, origin xyz=0 0 0.14 rpy=3.141592653589793 0 0
