Commit message: Added a script to show the camera API.

File: coffee/models/vendor/robot_arms/franka_emika/panda_description/panda.urdf (robot description, URDF)
Before this commit: robot panda, 10 links, 9 joints
Joints:
- joint ee_fixed_joint: origin xyz=0.0 0.0 0. rpy=0.0 0.0 0.0 -> xyz=0.0 0.0 0. rpy=0 3.141592653589793 3.141592653589793
