Commit message: Joint limiting the UR5 + nit fixes.

File: coffee/models/vendor/end_effectors/onrobot/rg2_description/model.urdf (robot description, URDF)
Before this commit: robot rg2, 7 links, 6 joints
Links:
- added link pinch_site, mass 0.0; collision box size=0 0 0; visual box size=0.01 0.01 0.01
Joints:
- added joint tcp_joint: type fixed, parent palm, child pinch_site, origin xyz=0 0 0.135 rpy=3.141592653589793 0 0

File: coffee/models/vendor/robot_arms/universal_robot/ur5_description/ur5.urdf (robot description, URDF)
Before this commit: robot universal_robot, 8 links, 7 joints
Joints:
- joint shoulder_lift_joint: limit lower=-6.28318530718 upper=6.28318530718 effort=150.0 velocity=3.15 -> lower=-3.14159265359 upper=3.14159265359 effort=150.0 velocity=3.15
- joint shoulder_pan_joint: limit lower=-6.28318530718 upper=6.28318530718 effort=150.0 velocity=3.15 -> lower=-3.14159265359 upper=3.14159265359 effort=150.0 velocity=3.15
- joint wrist_1_joint: limit lower=-6.28318530718 upper=6.28318530718 effort=28.0 velocity=3.2 -> lower=-3.14159265359 upper=3.14159265359 effort=28.0 velocity=3.2
- joint wrist_2_joint: limit lower=-6.28318530718 upper=6.28318530718 effort=28.0 velocity=3.2 -> lower=-3.14159265359 upper=3.14159265359 effort=28.0 velocity=3.2
- joint wrist_3_joint: limit lower=-6.28318530718 upper=6.28318530718 effort=28.0 velocity=3.2 -> lower=-3.14159265359 upper=3.14159265359 effort=28.0 velocity=3.2
